File: docs/MPPT_navitas/SM72442 breakout board/SM72442 Breakout Board/SM72442 Breakout Board.kicad_pcb (KiCad board)
At the start: 2 copper layers, 3 parts, among them J1 Conn_01x14_Male, J2 Conn_01x14_Male, U1 SM72442MT_NOPB

Commit message: update
Parts:
- J1, J2: footprint Connector_PinHeader_2.54mm:PinHeader_1x14_P2.54mm_Vertical -> Connector_PinHeader_2.54mm:PinHeader_1x13_P2.54mm_Vertical
- moved J2 27.7 mm to (147.3, 118.1), turned to 0 degrees
- moved U1 7.41 mm to (138.4, 135.9)
- moved J1 6.48 mm to (129.5, 118.1)
Connections:
- J2 pad 1: /AVIN -> /PM
- J2 pad 10: /LIB -> /AIIN
- J2 pad 11: /HIB -> /A4
- J2 pad 12: /HIA -> /AVOUT
- J2 pad 13: /LIA -> /A2
- J2 pad 2: /A2 -> /LIA
- J2 pad 3: /AVOUT -> /HIA
- J2 pad 4: /A4 -> /HIB
- J2 pad 5: /AIIN -> /LIB
- J2 pad 6: /A6 -> /NC4
- J2 pad 7: /AIOUT -> /I2C2
- J2 pad 8: /I2C2 -> /AIOUT
- J2 pad 9: /NC4 -> /A6
Routing:
- net /PM: track 17.6 -> 0.00 mm
- net /LIA: track 16.9 -> 0.00 mm
- net /A0: track 16.4 -> 0.00 mm
- net /HIA: track 15.4 -> 0.00 mm
- net /AVIN: track 15.1 -> 0.00 mm
- net /A2: track 14.4 -> 0.00 mm
- net /VSSA: track 14.9 -> 1.27 mm
- net /AVOUT: track 13.6 -> 0.00 mm
- net /HIB: track 13.1 -> 0.00 mm
- net /LIB: track 12.3 -> 0.00 mm
- net /A4: track 12.0 -> 0.00 mm
- net /NC4: track 11.5 -> 0.00 mm
- net /AIIN: track 11.3 -> 0.00 mm
- net /I2C2: track 10.8 -> 0.00 mm
- net /A6: track 10.5 -> 0.00 mm
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
Commit message: update on PCB
Parts:
- J1, J2: footprint Connector_PinHeader_2.54mm:PinHeader_1x13_P2.54mm_Vertical -> Connector_PinHeader_2.54mm:PinHeader_1x14_P2.54mm_Vertical
- moved U1 1.27 mm to (138.4, 134.6)
Routing:
- net /A0: track 0.00 -> 14.8 mm
- net /PM: track 0.00 -> 14.8 mm
- net /AVIN: track 0.00 -> 14.8 mm
- net /A2: track 0.00 -> 13.3 mm
- net /LIA: track 0.00 -> 13.3 mm
- net /VSSA: track 1.27 -> 13.3 mm
- net /AVOUT: track 0.00 -> 11.5 mm
- net /HIA: track 0.00 -> 11.5 mm
- net /HIB: track 0.00 -> 9.57 mm
- net /A4: track 0.00 -> 9.57 mm
- net /LIB: track 0.00 -> 7.98 mm
- net /AIIN: track 0.00 -> 7.98 mm
- net /NC4: track 0.00 -> 7.19 mm
- net /A6: track 0.00 -> 7.19 mm
- net /I2C2: track 0.00 -> 6.41 mm
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Other:
- board outline added: 22.9 x 38.1 mm
- rule pad_to_mask_clearance: 0 -> 0.05
- board text added: "SM 72442 board"
