File: docs/MPPT_navitas/MPPT_Apollo_noSTM/MPPT_Apollo_noSTM.kicad_pcb (KiCad board)
At the start: 2 copper layers, 160 parts, among them J10 Conn_01x03_Male, J15 Conn_01x03_Female, J6 PV, J7 BAT, Q1 2N7002, Q2 Q_NPN_BCE, Q3 2N7002, Q4 2N7002, Q5 2N7002, Q6 2N7002, U10 Driver_FET_SM72295MA_Navitas, U10A1 SM72375, U10B1 SM72375, U11A1 MCP602-I_SN, U11B1 MCP602-I_SN, U12 INA199A1DCKR_NAVITAS, U13 INA199A1DCKR_NAVITAS, U8 SM72442MT_NOPB_Navitas

Commit message: PCB update
Parts:
- moved C65 68.9 mm to (120.9, 62.0), turned to 90 degrees
- moved C67 64.7 mm to (119.4, 62.0), turned to 90 degrees
- moved C59 63.9 mm to (125.5, 62.0), turned to 90 degrees
- moved C53 63.4 mm to (128.5, 62.0), turned to 90 degrees
- moved C62 61.6 mm to (124.0, 61.9), turned to 90 degrees
- moved C55 61.4 mm to (127.0, 62.0), turned to 90 degrees
- moved C63 61.2 mm to (122.4, 61.9), turned to 90 degrees
- moved C51 57.7 mm to (130.0, 62.0), turned to 90 degrees
